Commit message: modify caster mass

File: vicpinky_description/urdf/robot_core.xacro (robot description, xacro)
@@ -14,5 +14,5 @@
     <xacro:property name="wheel_mass" value="0.05"/>
     <xacro:property name="caster_wheel_radius" value="${wheel_diameter/2}"/>
-    <xacro:property name="caster_wheel_mass" value="1.0"/>
+    <xacro:property name="caster_wheel_mass" value="2.0"/>
     <xacro:property name="chassis_x_offset" value="${-chassis_length/2+0.1}"/>
     <material name="white">

Commit message: modify caster mass

File: vicpinky_description/urdf/robot_core.xacro (robot description, xacro)
@@ -14,5 +14,5 @@
     <xacro:property name="wheel_mass" value="0.05"/>
     <xacro:property name="caster_wheel_radius" value="${wheel_diameter/2}"/>
-    <xacro:property name="caster_wheel_mass" value="2.0"/>
+    <xacro:property name="caster_wheel_mass" value="3.0"/>
     <xacro:property name="chassis_x_offset" value="${-chassis_length/2+0.1}"/>
     <material name="white">

Commit message: update gazebo

File: vicpinky_description/urdf/robot_core.xacro (robot description, xacro)
@@ -19,4 +19,7 @@
         <color rgba="1 1 1 1" />
     </material>
+    <material name="gray">
+        <color rgba="0.2 0.2 0.2 1" />
+    </material>
     <material name="black">
         <color rgba="0 0 0 1"/>
@@ -35,5 +38,5 @@
                 <box size="${pillar_size} ${pillar_size} ${pillar_height}"/>
             </geometry>
-            <material name="white"/>
+            <material name="gray"/>
         </visual>
         <collision>
@@ -53,5 +56,5 @@
                 <box size="${chassis_length} ${chassis_width} ${chassis_height}"/>
             </geometry>
-            <material name="white"/>
+            <material name="gray"/>
         </visual>
         <collision>
@@ -73,5 +76,5 @@
                 <box size="${chassis_length} ${chassis_width} 0.03"/>
             </geometry>
-            <material name="white"/>
+            <material name="gray"/>
         </visual>
         <collision>
@@ -150,5 +153,5 @@
                 <sphere radius="${caster_wheel_radius}"/>
             </geometry>
-            <material name="white"/>
+            <material name="gray"/>
         </visual>
         <collision>
@@ -173,5 +176,5 @@
                 <sphere radius="${caster_wheel_radius}"/>
             </geometry>
-            <material name="white"/>
+            <material name="gray"/>
         </visual>
         <collision>

Commit message: update urdf

File: vicpinky_description/urdf/robot_core.xacro (robot description, xacro)
@@ -188,34 +188,4 @@
         </xacro:inertial_sphere>
     </link>
-    <link name="${prefix}front_camera_mount">
-        <visual>
-            <origin xyz="0 0 0" rpy="0 0 0"/>
-            <geometry>
-                <mesh filename="package://vicpinky_description/meshes/visual/camera.dae" scale="1 1 1"/>
-            </geometry>
-        </visual>
-        <collision>
-            <origin xyz="0 0 0" rpy="0 0 0"/>
-            <geometry>
-                <mesh filename="package://vicpinky_description/meshes/collision/camera.stl" scale="1 1 1"/>
-            </geometry>
-        </collision>
-        <inertial>
-            <origin xyz="0.005 0 0.013" rpy="0 0 0"/>
-            <mass value="0.050000"/>
-            <inertia ixx="0.000005" ixy="0" ixz="-0.000001" iyy="0.000004" iyz="0" izz="0.000003"/>
-        </inertial>
-    </link>
-    <joint name="${prefix}front_camera_mount_fixed_joint" type="fixed">
-        <parent link="${prefix}base_link"/>
-        <child link="${prefix}front_camera_mount"/>
-        <origin xyz="0.05 -0.001 0.028" rpy="0 0 0"/>
-    </joint>
-    <link name="${prefix}camera_link"/>
-    <joint name="${prefix}camera_link_fixed_joint" type="fixed">
-        <parent link="${prefix}front_camera_mount"/>
-        <child link="${prefix}camera_link"/>
-        <origin xyz="0.001 0 0.003" rpy="-${pi/2} 0 -${pi/2}"/>
-    </joint>
     <link name="${prefix}lidar_mount">
         <visual>

Commit message: feat: change lidar tf

File: vicpinky_description/urdf/robot_core.xacro (robot description, xacro)
@@ -227,5 +227,5 @@
         <parent link="${prefix}base_link"/>
         <child link="${prefix}lidar_mount"/>
-        <origin xyz="0 0 0.52" rpy="${pi} 0 0"/>
+        <origin xyz="0 0 0.18" rpy="0 0 0"/>
     </joint>
     <link name="${prefix}laser_link"/>
