Commit message: add namespace

File: vicpinky_description/urdf/gazebo_control.xacro (robot description, xacro)
@@ -1,8 +1,10 @@
 <?xml version="1.0"?>
 <robot xmlns:xacro="http://www.ros.org/wiki/xacro">
+    <xacro:arg name="namespace" default=""/>
+    <xacro:property name="prefix" value="$(arg namespace)"/>
     <gazebo>
         <plugin filename="gz-sim-diff-drive-system" name="gz::sim::systems::DiffDrive">
-            <left_joint>left_wheel_joint</left_joint>
-            <right_joint>right_wheel_joint</right_joint>
+            <left_joint>${prefix}left_wheel_joint</left_joint>
+            <right_joint>${prefix}right_wheel_joint</right_joint>
             <wheel_separation>0.425</wheel_separation>
             <wheel_radius>0.0825</wheel_radius>
@@ -11,15 +13,15 @@
             <min_acceleration>-2.0</min_acceleration>
             <max_acceleration>2.0</max_acceleration>
-            <topic>cmd_vel</topic>
-            <odom_topic>odom</odom_topic>
-            <frame_id>odom</frame_id>
-            <child_frame_id>base_footprint</child_frame_id>
+            <topic>${prefix}cmd_vel</topic>
+            <odom_topic>${prefix}odom</odom_topic>
+            <frame_id>${prefix}odom</frame_id>
+            <child_frame_id>${prefix}base_footprint</child_frame_id>
             <odom_publisher_frequency>30</odom_publisher_frequency>
             <tf_topic>/tf</tf_topic>
         </plugin>
         <plugin filename="gz-sim-joint-state-publisher-system" name="gz::sim::systems::JointStatePublisher">
-            <topic>joint_states</topic>
-            <joint_name>left_wheel_joint</joint_name>
-            <joint_name>right_wheel_joint</joint_name>
+            <topic>${prefix}joint_states</topic>
+            <joint_name>${prefix}left_wheel_joint</joint_name>
+            <joint_name>${prefix}right_wheel_joint</joint_name>
         </plugin>
     </gazebo>

File: vicpinky_description/urdf/lidar.xacro (robot description, xacro)
@@ -1,5 +1,7 @@
 <?xml version="1.0"?>
 <robot xmlns:xacro="http://www.ros.org/wiki/xacro" >
-    <gazebo reference="laser_link">
+    <xacro:arg name="namespace" default=""/>
+    <xacro:property name="prefix" value="$(arg namespace)"/>
+    <gazebo reference="${prefix}laser_link">
         <sensor name="laser" type="gpu_lidar">
             <always_on>true</always_on>
@@ -7,6 +9,6 @@
             <pose> 0 0 0 0 0 0 </pose>
             <update_rate>5</update_rate>
-            <topic>scan</topic>
-            <gz_frame_id>laser_link</gz_frame_id>
+            <topic>${prefix}scan</topic>
+            <gz_frame_id>${prefix}laser_link</gz_frame_id>
             <lidar>
                 <scan>

File: vicpinky_description/urdf/robot_core.xacro (robot description, xacro)
@@ -1,4 +1,6 @@
 <?xml version="1.0"?>
 <robot name="pinky" xmlns:xacro="http://www.ros.org/wiki/xacro">
+    <xacro:arg name="namespace" default=""/>
+    <xacro:property name="prefix" value="$(arg namespace)"/>
     <xacro:property name="wheel_separation" value="0.475"/>
     <xacro:property name="wheel_diameter" value="0.065"/>
@@ -12,5 +14,5 @@
     <xacro:property name="wheel_mass" value="0.05"/>
     <xacro:property name="caster_wheel_radius" value="${wheel_diameter/2}"/>
-    <xacro:property name="caster_wheel_mass" value="2.0"/>
+    <xacro:property name="caster_wheel_mass" value="1.0"/>
     <xacro:property name="chassis_x_offset" value="${-chassis_length/2+0.1}"/>
     <material name="white">
@@ -45,5 +47,5 @@
         </xacro:inertial_box>
     </xacro:macro>
-    <link name="base_link">
+    <link name="${prefix}base_link">
         <visual>
             <origin xyz="${chassis_x_offset} 0 ${chassis_height/2-0.02}" rpy="0 0 0"/>
@@ -83,17 +85,17 @@
         </xacro:inertial_box>
     </link>
-    <link name="base_footprint"/>
-    <joint name="base_link_fixed_joint" type="fixed">
-        <parent link="base_footprint"/>
-        <child link="base_link"/>
+    <link name="${prefix}base_footprint"/>
+    <joint name="${prefix}base_link_fixed_joint" type="fixed">
+        <parent link="${prefix}base_footprint"/>
+        <child link="${prefix}base_link"/>
         <origin xyz="0 0 ${wheel_diameter/2}" rpy="0 0 0"/>
     </joint>
-    <joint name="left_wheel_joint" type="continuous">
-        <parent link="base_link"/>
-        <child link="left_wheel"/>
+    <joint name="${prefix}left_wheel_joint" type="continuous">
+        <parent link="${prefix}base_link"/>
+        <child link="${prefix}left_wheel"/>
         <origin xyz="0 ${wheel_separation/2} 0" rpy="-${pi/2} 0 0"/>
         <axis xyz="0 0 1"/>
     </joint>
-    <link name="left_wheel">
+    <link name="${prefix}left_wheel">
         <visual>
             <origin xyz="0 0 0" rpy="0 0 0"/>
@@ -113,11 +115,11 @@
         </xacro:inertial_cylinder>
     </link>
-    <joint name="right_wheel_joint" type="continuous">
-        <parent link="base_link"/>
-        <child link="right_wheel"/>
+    <joint name="${prefix}right_wheel_joint" type="continuous">
+        <parent link="${prefix}base_link"/>
+        <child link="${prefix}right_wheel"/>
         <origin xyz="0 ${-1 * wheel_separation/2} 0" rpy="${pi/2} 0 0"/>
         <axis xyz="0 0 -1"/>
     </joint>
-    <link name="right_wheel">
+    <link name="${prefix}right_wheel">
         <visual>
             <origin xyz="0 0 0" rpy="0 0 0"/>
@@ -137,10 +139,10 @@
         </xacro:inertial_cylinder>
     </link>
-    <joint name="left_caster_joint" type="fixed">
-        <parent link="base_link"/>
-        <child link="left_caster"/>
+    <joint name="${prefix}left_caster_joint" type="fixed">
+        <parent link="${prefix}base_link"/>
+        <child link="${prefix}left_caster"/>
         <origin xyz="${-chassis_length/2-0.1} ${chassis_width/2-0.1} ${-2*caster_wheel_radius+0.015}" rpy="0 0 0"/>
     </joint>
-    <link name="left_caster">
+    <link name="${prefix}left_caster">
       <visual>
             <origin xyz="0 0 0" rpy="0 0 0"/>
@@ -160,10 +162,10 @@
         </xacro:inertial_sphere>
     </link>
-    <joint name="right_caster_joint" type="fixed">
-        <parent link="base_link"/>
-        <child link="right_caster"/>
+    <joint name="${prefix}right_caster_joint" type="fixed">
+        <parent link="${prefix}base_link"/>
+        <child link="${prefix}right_caster"/>
         <origin xyz="${-chassis_length/2-0.1} ${-chassis_width/2+0.1} ${-2*caster_wheel_radius+0.015}" rpy="0 0 0"/>
     </joint>
-    <link name="right_caster">
+    <link name="${prefix}right_caster">
       <visual>
             <origin xyz="0 0 0" rpy="0 0 0"/>
@@ -183,5 +185,5 @@
         </xacro:inertial_sphere>
     </link>
-    <link name="front_camera_mount">
+    <link name="${prefix}front_camera_mount">
         <visual>
             <origin xyz="0 0 0" rpy="0 0 0"/>
@@ -202,16 +204,16 @@
         </inertial>
     </link>
-    <joint name="front_camera_mount_fixed_joint" type="fixed">
-        <parent link="base_link"/>
-        <child link="front_camera_mount"/>
+    <joint name="${prefix}front_camera_mount_fixed_joint" type="fixed">
+        <parent link="${prefix}base_link"/>
+        <child link="${prefix}front_camera_mount"/>
         <origin xyz="0.05 -0.001 0.028" rpy="0 0 0"/>
     </joint>
-    <link name="camera_link"/>
-    <joint name="camera_link_fixed_joint" type="fixed">
-        <parent link="front_camera_mount"/>
-        <child link="camera_link"/>
+    <link name="${prefix}camera_link"/>
+    <joint name="${prefix}camera_link_fixed_joint" type="fixed">
+        <parent link="${prefix}front_camera_mount"/>
+        <child link="${prefix}camera_link"/>
         <origin xyz="0.001 0 0.003" rpy="-${pi/2} 0 -${pi/2}"/>
     </joint>
-    <link name="lidar_mount">
+    <link name="${prefix}lidar_mount">
         <visual>
             <origin xyz="0 0 0" rpy="0 0 0"/>
@@ -249,13 +251,13 @@
         </xacro:inertial_box>
     </link>
-    <joint name="lidar_mount_fixed_joint" type="fixed">
-        <parent link="base_link"/>
-        <child link="lidar_mount"/>
+    <joint name="${prefix}lidar_mount_fixed_joint" type="fixed">
+        <parent link="${prefix}base_link"/>
+        <child link="${prefix}lidar_mount"/>
         <origin xyz="0 0 0.52" rpy="${pi} 0 0"/>
     </joint>
-    <link name="laser_link"/>
-    <joint name="laser_link_fixed_joint" type="fixed">
-        <parent link="lidar_mount"/>
-        <child link="laser_link"/>
+    <link name="${prefix}laser_link"/>
+    <joint name="${prefix}laser_link_fixed_joint" type="fixed">
+        <parent link="${prefix}lidar_mount"/>
+        <child link="${prefix}laser_link"/>
         <origin xyz="0.0 0 0.03" rpy="0 0 ${pi}"/>
     </joint>

File: vicpinky_description/urdf/robot_gazebo.xacro (robot description, xacro)
@@ -1,24 +1,26 @@
 <?xml version="1.0"?>
 <robot name="pinky" xmlns:xacro="http://www.ros.org/wiki/xacro">
-    <gazebo reference="left_wheel">
+    <xacro:arg name="namespace" default=""/>
+    <xacro:property name="prefix" value="$(arg namespace)"/>
+    <gazebo reference="${prefix}left_wheel">
         <selfCollide>false</selfCollide>
         <mu1 value="1.2" />
         <mu2 value="1.2" />
     </gazebo>
-    <gazebo reference="right_wheel">
+    <gazebo reference="${prefix}right_wheel">
         <selfCollide>false</selfCollide>
         <mu1 value="1.2" />
         <mu2 value="1.2" />
     </gazebo>
-    <gazebo reference="base_link">
+    <gazebo reference="${prefix}base_link">
         <selfCollide>false</selfCollide>
         <mu1 value="0.01" />
         <mu2 value="0.01" />
     </gazebo>
-    <gazebo reference="left_caster">
+    <gazebo reference="${prefix}left_caster">
       <mu1 value="0.01" />
       <mu2 value="0.01" />
     </gazebo>
-    <gazebo reference="right_caster">
+    <gazebo reference="${prefix}right_caster">
       <mu1 value="0.01" />
       <mu2 value="0.01" />

Commit message: feat(vicpinky): update version to v2.0.0

File: vicpinky_description/urdf/gazebo_control.xacro (robot description, xacro)
@@ -7,5 +7,5 @@
             <left_joint>${prefix}left_wheel_joint</left_joint>
             <right_joint>${prefix}right_wheel_joint</right_joint>
-            <wheel_separation>0.425</wheel_separation>
+            <wheel_separation>0.3788</wheel_separation>
             <wheel_radius>0.0825</wheel_radius>
             <min_velocity>-1.0</min_velocity>

File: vicpinky_description/urdf/robot_core.xacro (robot description, xacro)
@@ -1,19 +1,22 @@
 <?xml version="1.0"?>
-<robot name="pinky" xmlns:xacro="http://www.ros.org/wiki/xacro">
+<robot name="vicpinky" xmlns:xacro="http://www.ros.org/wiki/xacro">
     <xacro:arg name="namespace" default=""/>
     <xacro:property name="prefix" value="$(arg namespace)"/>
-    <xacro:property name="wheel_separation" value="0.475"/>
-    <xacro:property name="wheel_diameter" value="0.065"/>
     <xacro:include filename="inertial_macros.xacro"/>
+    <xacro:property name="wheel_separation" value="0.4288"/>
     <xacro:property name="chassis_length" value="0.6"/>
-    <xacro:property name="chassis_width" value="0.4"/>
-    <xacro:property name="chassis_height" value="0.14"/>
+    <xacro:property name="chassis_width" value="0.5"/>
+    <xacro:property name="chassis_height" value="0.128"/>
     <xacro:property name="chassis_mass" value="50.0"/>
+    <xacro:property name="chassis_z_offset" value="0.087"/>
     <xacro:property name="wheel_radius" value="0.0825"/>
     <xacro:property name="wheel_thickness" value="0.05"/>
     <xacro:property name="wheel_mass" value="0.05"/>
-    <xacro:property name="caster_wheel_radius" value="${wheel_diameter/2}"/>
+    <xacro:property name="caster_wheel_radius" value="${chassis_z_offset/2}"/>
     <xacro:property name="caster_wheel_mass" value="3.0"/>
-    <xacro:property name="chassis_x_offset" value="${-chassis_length/2+0.1}"/>
+    <xacro:property name="caster_x_inset" value="0.056"/>
+    <xacro:property name="caster_y_inset" value="0.156"/>
+    <xacro:property name="caster_x_offset" value="${chassis_length/2 - caster_x_inset}"/>
+    <xacro:property name="caster_y_offset" value="${chassis_width/2 - caster_y_inset}"/>
     <material name="white">
         <color rgba="1 1 1 1" />
@@ -28,36 +31,14 @@
         <color rgba="0 0 1 1"/>
     </material>
-    <xacro:property name="pillar_mass" value="0.1"/>
-    <xacro:property name="pillar_size" value="0.03"/>
-    <xacro:property name="pillar_height" value="0.5"/>
-    <xacro:property name="pillar_inset" value="0.015"/>
-    <xacro:macro name="pillar" params="prefix x y">
+    <link name="${prefix}base_link">
         <visual>
-            <origin xyz="${x} ${y} ${chassis_height + pillar_height/2 - 0.02}" rpy="0 0 0"/>
+            <origin xyz="0 0 0" rpy="0 0 0"/>
             <geometry>
-                <box size="${pillar_size} ${pillar_size} ${pillar_height}"/>
+                <mesh filename="package://vicpinky_description/meshes/visual/base_link.stl" scale="1 1 1"/>
             </geometry>
             <material name="gray"/>
         </visual>
         <collision>
-            <origin xyz="${x} ${y} ${chassis_height + pillar_height/2 - 0.02}" rpy="0 0 0"/>
-            <geometry>
-                <box size="${pillar_size} ${pillar_size} ${pillar_height}"/>
-            </geometry>
-        </collision>
-        <xacro:inertial_box mass="${pillar_mass}" x="${pillar_size}" y="${pillar_size}" z="${pillar_height}">
-            <origin xyz="${x} ${y} ${chassis_height + pillar_height/2 - 0.02}" rpy="0 0 0"/>
-        </xacro:inertial_box>
-    </xacro:macro>
-    <link name="${prefix}base_link">
-        <visual>
-            <origin xyz="${chassis_x_offset} 0 ${chassis_height/2-0.02}" rpy="0 0 0"/>
-            <geometry>
-                <box size="${chassis_length} ${chassis_width} ${chassis_height}"/>
-            </geometry>
-            <material name="gray"/>
-        </visual>
-        <collision>
-            <origin xyz="${chassis_x_offset} 0 ${chassis_height/2-0.02}" rpy="0 0 0"/>
+            <origin xyz="0 0 ${chassis_height/2-0.02}" rpy="0 0 0"/>
             <geometry>
                 <box size="${chassis_length} ${chassis_width} ${chassis_height}"/>
@@ -67,24 +48,4 @@
             <origin xyz="0 0 0" rpy="0 0 0"/>
         </xacro:inertial_box>
-        <xacro:pillar prefix="front_left"  x="${chassis_x_offset + chassis_length/2 - pillar_inset}" y="${chassis_width/2 - pillar_inset}"/>
-        <xacro:pillar prefix="front_right" x="${chassis_x_offset + chassis_length/2 - pillar_inset}" y="-${chassis_width/2 - pillar_inset}"/>
-        <xacro:pillar prefix="rear_left"   x="${chassis_x_offset - chassis_length/2 + pillar_inset}" y="${chassis_width/2 - pillar_inset}"/>
-        <xacro:pillar prefix="rear_right"  x="${chassis_x_offset - chassis_length/2 + pillar_inset}" y="-${chassis_width/2 - pillar_inset}"/>
-        <visual>
-            <origin xyz="${chassis_x_offset} 0 ${chassis_height/2 + pillar_height + 0.03}" rpy="0 0 0"/>
-            <geometry>
-                <box size="${chassis_length} ${chassis_width} 0.03"/>
-            </geometry>
-            <material name="gray"/>
-        </visual>
-        <collision>
-            <origin xyz="${chassis_x_offset} 0 ${chassis_height/2 + pillar_height + 0.03}" rpy="0 0 0"/>
-            <geometry>
-                <box size="${chassis_length} ${chassis_width} 0.03"/>
-            </geometry>
-        </collision>
-        <xacro:inertial_box mass="${chassis_mass}" x="${chassis_length}" y="${chassis_width}" z="0.03">
-            <origin xyz="${chassis_x_offset} 0 ${chassis_height/2 + pillar_height + 0.03}" rpy="0 0 0"/>
-        </xacro:inertial_box>
     </link>
     <link name="${prefix}base_footprint"/>
@@ -92,17 +53,17 @@
         <parent link="${prefix}base_footprint"/>
         <child link="${prefix}base_link"/>
-        <origin xyz="0 0 ${wheel_diameter/2}" rpy="0 0 0"/>
+        <origin xyz="0 0 ${chassis_z_offset}" rpy="0 0 0"/>
     </joint>
     <joint name="${prefix}left_wheel_joint" type="continuous">
         <parent link="${prefix}base_link"/>
         <child link="${prefix}left_wheel"/>
-        <origin xyz="0 ${wheel_separation/2} 0" rpy="-${pi/2} 0 0"/>
+        <origin xyz="0 ${wheel_separation/2} -0.0048" rpy="-${pi/2} 0 0"/>
         <axis xyz="0 0 1"/>
     </joint>
     <link name="${prefix}left_wheel">
         <visual>
-            <origin xyz="0 0 0" rpy="0 0 0"/>
+            <origin xyz="0 0 0" rpy="0 ${-pi/2} 0"/>
             <geometry>
-                <cylinder radius="${wheel_radius}" length="${wheel_thickness}"/>
+                <mesh filename="package://vicpinky_description/meshes/visual/wheel.stl" scale="1 1 1"/>
             </geometry>
             <material name="black"/>
@@ -121,12 +82,12 @@
         <parent link="${prefix}base_link"/>
         <child link="${prefix}right_wheel"/>
-        <origin xyz="0 ${-1 * wheel_separation/2} 0" rpy="${pi/2} 0 0"/>
+        <origin xyz="0 ${-1 * wheel_separation/2} -0.0048" rpy="${pi/2} 0 0"/>
         <axis xyz="0 0 -1"/>
     </joint>
     <link name="${prefix}right_wheel">
         <visual>
-            <origin xyz="0 0 0" rpy="0 0 0"/>
+            <origin xyz="0 0.0 0.0" rpy="0 ${-pi/2} 0"/>
             <geometry>
-                <cylinder radius="${wheel_radius}" length="${wheel_thickness}"/>
+                <mesh filename="package://vicpinky_description/meshes/visual/wheel.stl" scale="1 1 1"/>
             </geometry>
             <material name="black"/>
@@ -142,50 +103,33 @@
         </xacro:inertial_cylinder>
     </link>
-    <joint name="${prefix}left_caster_joint" type="fixed">
-        <parent link="${prefix}base_link"/>
-        <child link="${prefix}left_caster"/>
-        <origin xyz="${-chassis_length/2-0.1} ${chassis_width/2-0.1} ${-2*caster_wheel_radius+0.015}" rpy="0 0 0"/>
-    </joint>
-    <link name="${prefix}left_caster">
-      <visual>
-            <origin xyz="0 0 0" rpy="0 0 0"/>
-            <geometry>
-                <sphere radius="${caster_wheel_radius}"/>
-            </geometry>
-            <material name="gray"/>
-        </visual>
-        <collision>
-            <origin xyz="0 0 0" rpy="0 0 0"/>
-            <geometry>
-                <sphere radius="${caster_wheel_radius}"/>
-            </geometry>
-        </collision>
-        <xacro:inertial_sphere mass="${caster_wheel_mass}" radius="${caster_wheel_radius}">
-            <origin xyz="0 0 0" rpy="0 0 0"/>
-        </xacro:inertial_sphere>
-    </link>
-    <joint name="${prefix}right_caster_joint" type="fixed">
-        <parent link="${prefix}base_link"/>
-        <child link="${prefix}right_caster"/>
-        <origin xyz="${-chassis_length/2-0.1} ${-chassis_width/2+0.1} ${-2*caster_wheel_radius+0.015}" rpy="0 0 0"/>
-    </joint>
-    <link name="${prefix}right_caster">
-      <visual>
-            <origin xyz="0 0 0" rpy="0 0 0"/>
-            <geometry>
-                <sphere radius="${caster_wheel_radius}"/>
-            </geometry>
-            <material name="gray"/>
-        </visual>
-        <collision>
-            <origin xyz="0 0 0" rpy="0 0 0"/>
-            <geometry>
-                <sphere radius="${caster_wheel_radius}"/>
-            </geometry>
-        </collision>
-        <xacro:inertial_sphere mass="${caster_wheel_mass}" radius="${caster_wheel_radius}">
-            <origin xyz="0 0 0" rpy="0 0 0"/>
-        </xacro:inertial_sphere>
-    </link>
+    <xacro:macro name="caster_wheel" params="suffix x_offset y_offset">
+        <joint name="${prefix}${suffix}_caster_joint" type="fixed">
+            <parent link="${prefix}base_link"/>
+            <child link="${prefix}${suffix}_caster"/>
+            <origin xyz="${x_offset} ${y_offset} ${-chassis_z_offset + caster_wheel_radius}" rpy="0 0 0"/>
+        </joint>
+        <link name="${prefix}${suffix}_caster">
+            <visual>
+                <origin xyz="0 0 ${caster_wheel_radius}" rpy="0 0 0"/>
+                <geometry>
+                    <mesh filename="package://vicpinky_description/meshes/visual/caster.stl" scale="1 1 1"/>
+                </geometry>
+                <material name="gray"/>
+            </visual>
+            <collision>
+                <origin xyz="0 0 0" rpy="0 0 0"/>
+                <geometry>
+                    <sphere radius="${caster_wheel_radius}"/>
+                </geometry>
+            </collision>
+            <xacro:inertial_sphere mass="${caster_wheel_mass}" radius="${caster_wheel_radius}">
+                <origin xyz="0 0 0" rpy="0 0 0"/>
+            </xacro:inertial_sphere>
+        </link>
+    </xacro:macro>
+    <xacro:caster_wheel suffix="front_left"  x_offset="${caster_x_offset}"  y_offset="${caster_y_offset}"/>
+    <xacro:caster_wheel suffix="front_right" x_offset="${caster_x_offset}"  y_offset="${-caster_y_offset}"/>
+    <xacro:caster_wheel suffix="rear_left"   x_offset="${-caster_x_offset}" y_offset="${caster_y_offset}"/>
+    <xacro:caster_wheel suffix="rear_right"  x_offset="${-caster_x_offset}" y_offset="${-caster_y_offset}"/>
     <link name="${prefix}lidar_mount">
         <visual>
@@ -194,5 +138,4 @@
                 <mesh filename="package://vicpinky_description/meshes/visual/lidar.dae" scale="1 1 1"/>
             </geometry>
-            <material name="blue"/>
         </visual>
         <collision>
@@ -207,25 +150,9 @@
             <inertia ixx="0.000058" ixy="0" ixz="0.000005" iyy="0.000099" iyz="0" izz="0.000103"/>
         </inertial>
-        <visual>
-            <origin xyz="0 0 -0.035" rpy="0 0 0"/>
-            <geometry>
-                <box size="0.07 0.07 0.07"/>
-            </geometry>
-            <material name="blue"/>
-        </visual>
-        <collision>
-            <origin xyz="0 0 -0.035" rpy="0 0 0"/>
-            <geometry>
-                <box size="0.07 0.07 0.07"/>
-            </geometry>
-        </collision>
-        <xacro:inertial_box mass="0.03" x="0.07" y="0.07" z="0.07">
-            <origin xyz="0 0 -0.035" rpy="0 0 0"/>
-        </xacro:inertial_box>
     </link>
     <joint name="${prefix}lidar_mount_fixed_joint" type="fixed">
         <parent link="${prefix}base_link"/>
         <child link="${prefix}lidar_mount"/>
-        <origin xyz="0 0 0.18" rpy="0 0 0"/>
+        <origin xyz="0.185 0.0 0.12" rpy="0 0 0"/>
     </joint>
     <link name="${prefix}laser_link"/>
